Commit message: dimension parameters to URDF

File: balboa_description/urdf/balboa.urdf.xacro (robot description, xacro)
@@ -3,4 +3,17 @@
   <xacro:include filename="$(find balboa_description)/urdf/common_properties.urdf.xacro"/>
   <xacro:include filename="$(find balboa_description)/urdf/wheel.urdf.xacro"/>
+  <xacro:property name="body_x" value="${0.5*cm2m}" />
+  <xacro:property name="body_y" value="${2*cm2m}" />
+  <xacro:property name="body_z" value="${5*cm2m}" />
+  <xacro:property name="wheel_radius" value="${1*cm2m}" />
+  <xacro:property name="wheel_width" value="${0.5*cm2m}" />
+  <xacro:property name="distance_between_wheels" value="${2*cm2m}" />
+  <link name="origin_link">
+  </link>
+  <joint name="origin_joint" type="fixed">
+    <origin xyz="0 0 ${wheel_radius}" rpy="0 0 0"/>
+    <parent link="origin_link"/>
+    <child link="base_link"/>
+  </joint>
   <!-- Create 3 base definition-->
   <link name="base_link">
@@ -17,5 +30,5 @@
       </geometry>
     </collision>
-    <xacro:inertial_cuboid mass="1.0" x="0.005" y="0.02" z="0.05"/>
+    <xacro:inertial_cuboid mass="1.0" x="${body_x}" y="${body_y}" z="${body_z}"/>
   </link>
   <!-- Wheels -->
@@ -25,10 +38,10 @@
   </gazebo>
   <!-- Left wheel -->
-  <xacro:wheel name="left" parent_link="base_link">
-    <origin xyz="0 0.0155 0" rpy="${pi/2} 0 0"/>
+  <xacro:wheel name="left" width="${wheel_width}" radius="${wheel_radius}" parent_link="base_link">
+    <origin xyz="0 ${(body_y+wheel_width)/2} 0" rpy="${pi/2} 0 0"/>
   </xacro:wheel>
   <!-- Right wheel -->
-  <xacro:wheel name="right" parent_link="base_link">
-    <origin xyz="0 -0.0155 0" rpy="${pi/2} 0 0"/>
+  <xacro:wheel name="right" width="${wheel_width}" radius="${wheel_radius}" parent_link="base_link">
+    <origin xyz="0 ${-(body_y+wheel_width)/2} 0" rpy="${pi/2} 0 0"/>
   </xacro:wheel>
 </robot>

File: balboa_description/urdf/wheel.urdf.xacro (robot description, xacro)
@@ -1,8 +1,5 @@
 <?xml version="1.0"?>
 <robot xmlns:xacro="http://ros.org/wiki/xacro">
-<xacro:macro name="wheel" params="name parent_link *origin">
-  <xacro:property name="mass"   value="0.2" />
-  <xacro:property name="radius" value="${1.5*cm2m}" />
-  <xacro:property name="width"  value="${1*cm2m}" />
+<xacro:macro name="wheel" params="name mass:=0.2 radius:=0.015 width:=0.01 parent_link *origin">
   <xacro:property name="wheel_link_name"  value="${name}_wheel"/>
   <xacro:property name="wheel_joint_name" value="${wheel_link_name}_joint"/>

Commit message: diffdrive controller and IMU

File: balboa_description/urdf/balboa.urdf.xacro (robot description, xacro)
@@ -7,8 +7,7 @@
   <xacro:property name="body_z" value="${5*cm2m}" />
   <xacro:property name="wheel_radius" value="${1*cm2m}" />
-  <xacro:property name="wheel_width" value="${0.5*cm2m}" />
-  <xacro:property name="distance_between_wheels" value="${2*cm2m}" />
-  <link name="origin_link">
-  </link>
+  <xacro:property name="wheel_width" value="${0.1*cm2m}" />
+  <xacro:property name="encoder_resolution" value="1440" />
+  <link name="origin_link" />
   <joint name="origin_joint" type="fixed">
     <origin xyz="0 0 ${wheel_radius}" rpy="0 0 0"/>
@@ -30,9 +29,35 @@
       </geometry>
     </collision>
-    <xacro:inertial_cuboid mass="1.0" x="${body_x}" y="${body_y}" z="${body_z}"/>
+    <xacro:inertial_cuboid_with_pose mass="1.0" x="${body_x}" y="${body_y}" z="${body_z}">
+      <!-- <origin xyz="${body_x/2} ${body_y/2} ${body_z/2}" /> -->
+      <origin xyz="0 0 0" />
+    </xacro:inertial_cuboid_with_pose>
   </link>
+  <!-- IMU -->
+  <gazebo reference="base_link">
+      <gravity>true</gravity>
+      <sensor name="imu_sensor" type="imu">
+        <always_on>true</always_on>
+        <update_rate>100</update_rate>
+        <visualize>true</visualize>
+        <topic>__default_topic__</topic>
+        <plugin filename="libgazebo_ros_imu_sensor.so" name="imu_plugin">
+          <topicName>imu</topicName>
+          <bodyName>base_link</bodyName>
+          <updateRateHZ>10.0</updateRateHZ>
+          <gaussianNoise>0.0</gaussianNoise>
+          <xyzOffset>0 0 0</xyzOffset>
+          <rpyOffset>0 0 0</rpyOffset>
+          <frameName>base_link</frameName>
+        </plugin>
+        <pose>0 0 0 0 0 0</pose>
+      </sensor>
+    </gazebo>
   <!-- Wheels -->
   <gazebo>
     <plugin name="gazebo_diffdrive" filename="libgazebo_ros_diffdrive_controller.so">
+      <wheel_radius>${wheel_radius}</wheel_radius>
+      <wheel_distance>${wheel_width + body_y}</wheel_distance>
+      <encoder_resolution>${encoder_resolution}</encoder_resolution>
     </plugin>
   </gazebo>
@@ -45,3 +70,18 @@
     <origin xyz="0 ${-(body_y+wheel_width)/2} 0" rpy="${pi/2} 0 0"/>
   </xacro:wheel>
+  <!-- Ground truth pose -->
+  <gazebo>
+    <plugin name="gazebo_ros_p3d_robot" filename="libgazebo_ros_p3d.so">
+      <ros>
+        <namespace>/</namespace>
+        <remapping>odom:=sim_ground_truth_pose</remapping>
+      </ros>
+      <body_name>origin_link</body_name>
+      <frame_name>world</frame_name>
+      <update_rate>62</update_rate>
+      <xyz_offset>0 0 0</xyz_offset>
+      <rpy_offset>0.0 0.0 0.0</rpy_offset>
+      <gaussian_noise>0.0</gaussian_noise>
+    </plugin>
+  </gazebo>
 </robot>

File: balboa_description/urdf/wheel.urdf.xacro (robot description, xacro)
@@ -35,14 +35,4 @@
     <material>Gazebo/DarkGrey</material>
   </gazebo>
-  <ros2_control name="${wheel_link_name}_controller" type="system">
-    <hardware>
-      <plugin>gazebo_ros2_control/GazeboSystem</plugin>
-    </hardware>
-    <joint name="${wheel_joint_name}">
-      <state_interface name="velocity" />
-      <state_interface name="position" />
-      <command_interface name="velocity" />
-    </joint>
-  </ros2_control>
 </xacro:macro>
 </robot>

Commit message: imu link

File: balboa_description/urdf/balboa.urdf.xacro (robot description, xacro)
@@ -34,6 +34,12 @@
     </xacro:inertial_cuboid_with_pose>
   </link>
+  <joint name="imu_joint" type="fixed">
+    <origin xyz="0 0 0" rpy="0 0 0"/>
+    <parent link="base_link"/>
+    <child link="imu_link"/>
+  </joint>
+  <link name="imu_link"/>
   <!-- IMU -->
-  <gazebo reference="base_link">
+  <gazebo reference="imu_link">
       <gravity>true</gravity>
       <sensor name="imu_sensor" type="imu">
@@ -44,10 +50,11 @@
         <plugin filename="libgazebo_ros_imu_sensor.so" name="imu_plugin">
           <topicName>imu</topicName>
-          <bodyName>base_link</bodyName>
+          <bodyName>imu_link</bodyName>
           <updateRateHZ>10.0</updateRateHZ>
           <gaussianNoise>0.0</gaussianNoise>
           <xyzOffset>0 0 0</xyzOffset>
           <rpyOffset>0 0 0</rpyOffset>
-          <frameName>base_link</frameName>
+          <frameName>imu_link</frameName>
+          <initialOrientationAsReference>true</initialOrientationAsReference>
         </plugin>
         <pose>0 0 0 0 0 0</pose>

Commit message: PID failing to keep upright

File: balboa_description/urdf/balboa.urdf.xacro (robot description, xacro)
@@ -4,12 +4,13 @@
   <xacro:include filename="$(find balboa_description)/urdf/wheel.urdf.xacro"/>
   <xacro:property name="body_x" value="${0.5*cm2m}" />
-  <xacro:property name="body_y" value="${2*cm2m}" />
-  <xacro:property name="body_z" value="${5*cm2m}" />
+  <xacro:property name="body_y" value="${3*cm2m}" />
+  <xacro:property name="body_z" value="${2*cm2m}" />
   <xacro:property name="wheel_radius" value="${1*cm2m}" />
+  <xacro:property name="wheel_z_offset" value="${0.5*cm2m}" />
   <xacro:property name="wheel_width" value="${0.1*cm2m}" />
   <xacro:property name="encoder_resolution" value="1440" />
   <link name="origin_link" />
   <joint name="origin_joint" type="fixed">
-    <origin xyz="0 0 ${wheel_radius}" rpy="0 0 0"/>
+    <origin xyz="0 0 ${wheel_radius - wheel_z_offset}" rpy="0 0 0"/>
     <parent link="origin_link"/>
     <child link="base_link"/>
@@ -30,6 +31,6 @@
     </collision>
     <xacro:inertial_cuboid_with_pose mass="1.0" x="${body_x}" y="${body_y}" z="${body_z}">
-      <!-- <origin xyz="${body_x/2} ${body_y/2} ${body_z/2}" /> -->
-      <origin xyz="0 0 0" />
+      <origin xyz="${body_x/2} ${body_y/2} ${body_z/2}" />
+      <!-- <origin xyz="0 0 0" /> -->
     </xacro:inertial_cuboid_with_pose>
   </link>
@@ -64,9 +65,9 @@
   <!-- Left wheel -->
   <xacro:wheel name="left" width="${wheel_width}" radius="${wheel_radius}" parent_link="base_link">
-    <origin xyz="0 ${(body_y+wheel_width)/2} 0" rpy="${pi/2} 0 0"/>
+    <origin xyz="0 ${(body_y+wheel_width)/2} ${wheel_z_offset}" rpy="${pi/2} 0 0"/>
   </xacro:wheel>
   <!-- Right wheel -->
   <xacro:wheel name="right" width="${wheel_width}" radius="${wheel_radius}" parent_link="base_link">
-    <origin xyz="0 ${-(body_y+wheel_width)/2} 0" rpy="${pi/2} 0 0"/>
+    <origin xyz="0 ${-(body_y+wheel_width)/2} ${wheel_z_offset}" rpy="${pi/2} 0 0"/>
   </xacro:wheel>
   <!-- Ground truth pose -->

Commit message: sort of working

File: balboa_description/urdf/balboa.urdf.xacro (robot description, xacro)
@@ -6,6 +6,9 @@
   <xacro:property name="body_y" value="${3*cm2m}" />
   <xacro:property name="body_z" value="${2*cm2m}" />
+  <xacro:property name="imu_x" value="${0.01*cm2m}" />
+  <xacro:property name="imu_y" value="${0.01*cm2m}" />
+  <xacro:property name="imu_z" value="${0.01*cm2m}" />
   <xacro:property name="wheel_radius" value="${1*cm2m}" />
-  <xacro:property name="wheel_z_offset" value="${0.5*cm2m}" />
+  <xacro:property name="wheel_z_offset" value="${0.0*cm2m}" />
   <xacro:property name="wheel_width" value="${0.1*cm2m}" />
   <xacro:property name="encoder_resolution" value="1440" />
@@ -19,5 +22,5 @@
   <link name="base_link">
     <visual>
-      <origin xyz="0 0 0" rpy="0 0 0"/>
+      <origin xyz="0 0 0" rpy="0 ${25*deg2rad} 0"/>
       <geometry>
         <mesh filename="file://$(find balboa_description)/meshes/body.stl" />
@@ -31,6 +34,6 @@
     </collision>
     <xacro:inertial_cuboid_with_pose mass="1.0" x="${body_x}" y="${body_y}" z="${body_z}">
-      <origin xyz="${body_x/2} ${body_y/2} ${body_z/2}" />
-      <!-- <origin xyz="0 0 0" /> -->
+      <!-- <origin xyz="${body_x/2} ${body_y/2} ${body_z/2}" /> -->
+      <origin xyz="0 0 0" />
     </xacro:inertial_cuboid_with_pose>
   </link>
@@ -40,5 +43,9 @@
     <child link="imu_link"/>
   </joint>
-  <link name="imu_link"/>
+  <link name="imu_link">
+    <xacro:inertial_cuboid_with_pose mass="0.05" x="${imu_x}" y="${imu_y}" z="${imu_z}">
+      <origin xyz="${imu_x/2} ${imu_y/2} ${imu_z/2}" />
+    </xacro:inertial_cuboid_with_pose>
+  </link>
   <!-- IMU -->
 <gazebo reference="imu_link">

Commit message: updates update rates

File: balboa_description/urdf/balboa.urdf.xacro (robot description, xacro)
@@ -10,7 +10,8 @@
   <xacro:property name="imu_z" value="${0.01*cm2m}" />
   <xacro:property name="wheel_radius" value="${1*cm2m}" />
-  <xacro:property name="wheel_z_offset" value="${0.0*cm2m}" />
+  <xacro:property name="wheel_z_offset" value="${0.5*cm2m}" />
   <xacro:property name="wheel_width" value="${0.1*cm2m}" />
   <xacro:property name="encoder_resolution" value="1440" />
+  <xacro:property name="vel_update_rate" value="100" />
   <link name="origin_link" />
   <joint name="origin_joint" type="fixed">
@@ -22,5 +23,5 @@
   <link name="base_link">
     <visual>
-      <origin xyz="0 0 0" rpy="0 ${25*deg2rad} 0"/>
+      <origin xyz="0 0 0" rpy="0 ${0*deg2rad} 0"/>
       <geometry>
         <mesh filename="file://$(find balboa_description)/meshes/body.stl" />
@@ -34,6 +35,6 @@
     </collision>
     <xacro:inertial_cuboid_with_pose mass="1.0" x="${body_x}" y="${body_y}" z="${body_z}">
-      <!-- <origin xyz="${body_x/2} ${body_y/2} ${body_z/2}" /> -->
-      <origin xyz="0 0 0" />
+      <origin xyz="${body_x/2} ${body_y/2} ${body_z/2}" />
+      <!-- <origin xyz="0 0 0" /> -->
     </xacro:inertial_cuboid_with_pose>
   </link>
@@ -68,13 +69,14 @@
       <wheel_distance>${wheel_width + body_y}</wheel_distance>
       <encoder_resolution>${encoder_resolution}</encoder_resolution>
+      <vel_update_rate>${vel_update_rate}</vel_update_rate>
     </plugin>
   </gazebo>
   <!-- Left wheel -->
   <xacro:wheel name="left" width="${wheel_width}" radius="${wheel_radius}" parent_link="base_link">
-    <origin xyz="0 ${(body_y+wheel_width)/2} ${wheel_z_offset}" rpy="${pi/2} 0 0"/>
+    <origin xyz="0 ${(body_y+wheel_width)/2} ${wheel_z_offset}" rpy="${-pi/2} 0 0"/>
   </xacro:wheel>
   <!-- Right wheel -->
   <xacro:wheel name="right" width="${wheel_width}" radius="${wheel_radius}" parent_link="base_link">
-    <origin xyz="0 ${-(body_y+wheel_width)/2} ${wheel_z_offset}" rpy="${pi/2} 0 0"/>
+    <origin xyz="0 ${-(body_y+wheel_width)/2} ${wheel_z_offset}" rpy="${-pi/2} 0 0"/>
   </xacro:wheel>
   <!-- Ground truth pose -->

File: balboa_description/urdf/wheel.urdf.xacro (robot description, xacro)
@@ -22,4 +22,12 @@
         <cylinder length="${width}" radius="${radius}"/>
       </geometry>
+      <surface>
+        <friction>
+          <ode>
+            <mu>1</mu>
+            <mu2>1</mu2>
+          </ode>
+        </friction>
+      </surface>
     </collision>
     <xacro:inertial_cylinder mass="${mass}" radius="${radius}"
@@ -27,10 +35,10 @@
   </link>
   <gazebo reference="${wheel_link_name}">
-    <mu1>1.0</mu1>
+    <!-- <mu1>1.0</mu1>
     <mu2>1.0</mu2>
     <kp>1000000.0</kp>
     <kd>100.0</kd>
     <minDepth>0.0001</minDepth>
-    <maxVel>1.0</maxVel>
+    <maxVel>1.0</maxVel> -->
     <material>Gazebo/DarkGrey</material>
   </gazebo>

Commit message: changes

File: balboa_description/urdf/balboa.urdf.xacro (robot description, xacro)
@@ -10,4 +10,5 @@
   <xacro:property name="imu_z" value="${0.01*cm2m}" />
   <xacro:property name="wheel_radius" value="${1*cm2m}" />
+  <xacro:property name="wheel_mass" value="0.5" />
   <xacro:property name="wheel_z_offset" value="${0.5*cm2m}" />
   <xacro:property name="wheel_width" value="${0.1*cm2m}" />
@@ -44,8 +45,9 @@
     <child link="imu_link"/>
   </joint>
+  <gazebo reference="imu_joint">
+    <preserveFixedJoint>true</preserveFixedJoint>
+  </gazebo>
   <link name="imu_link">
-    <xacro:inertial_cuboid_with_pose mass="0.05" x="${imu_x}" y="${imu_y}" z="${imu_z}">
-      <origin xyz="${imu_x/2} ${imu_y/2} ${imu_z/2}" />
-    </xacro:inertial_cuboid_with_pose>
+    <xacro:inertial_dummy />
   </link>
   <!-- IMU -->
@@ -73,9 +75,9 @@
   </gazebo>
   <!-- Left wheel -->
-  <xacro:wheel name="left" width="${wheel_width}" radius="${wheel_radius}" parent_link="base_link">
+  <xacro:wheel name="left" width="${wheel_width}" radius="${wheel_radius}" mass="${wheel_mass}" parent_link="base_link">
     <origin xyz="0 ${(body_y+wheel_width)/2} ${wheel_z_offset}" rpy="${-pi/2} 0 0"/>
   </xacro:wheel>
   <!-- Right wheel -->
-  <xacro:wheel name="right" width="${wheel_width}" radius="${wheel_radius}" parent_link="base_link">
+  <xacro:wheel name="right" width="${wheel_width}" radius="${wheel_radius}" mass="${wheel_mass}" parent_link="base_link">
     <origin xyz="0 ${-(body_y+wheel_width)/2} ${wheel_z_offset}" rpy="${-pi/2} 0 0"/>
   </xacro:wheel>

Commit message: pitch range from -180 to 180

File: balboa_description/urdf/balboa.urdf.xacro (robot description, xacro)
@@ -11,5 +11,5 @@
   <xacro:property name="wheel_radius" value="${1*cm2m}" />
   <xacro:property name="wheel_mass" value="0.5" />
-  <xacro:property name="wheel_z_offset" value="${0.5*cm2m}" />
+  <xacro:property name="wheel_z_offset" value="${0.0*cm2m}" />
   <xacro:property name="wheel_width" value="${0.1*cm2m}" />
   <xacro:property name="encoder_resolution" value="1440" />
@@ -36,6 +36,6 @@
     </collision>
     <xacro:inertial_cuboid_with_pose mass="1.0" x="${body_x}" y="${body_y}" z="${body_z}">
-      <origin xyz="${body_x/2} ${body_y/2} ${body_z/2}" />
-      <!-- <origin xyz="0 0 0" /> -->
+      <!-- <origin xyz="${body_x/2} ${body_y/2} ${body_z/2}" /> -->
+      <origin xyz="0 0 0" />
     </xacro:inertial_cuboid_with_pose>
   </link>

Commit message: slows down rates

File: balboa_description/urdf/balboa.urdf.xacro (robot description, xacro)
@@ -14,5 +14,5 @@
   <xacro:property name="wheel_width" value="${0.1*cm2m}" />
   <xacro:property name="encoder_resolution" value="1440" />
-  <xacro:property name="vel_update_rate" value="100" />
+  <xacro:property name="vel_update_rate" value="10" />
   <link name="origin_link" />
   <joint name="origin_joint" type="fixed">
@@ -36,6 +36,6 @@
     </collision>
     <xacro:inertial_cuboid_with_pose mass="1.0" x="${body_x}" y="${body_y}" z="${body_z}">
-      <!-- <origin xyz="${body_x/2} ${body_y/2} ${body_z/2}" /> -->
-      <origin xyz="0 0 0" />
+      <origin xyz="${body_x/2} ${body_y/2} ${body_z/2}" />
+      <!-- <origin xyz="0 0 0" /> -->
     </xacro:inertial_cuboid_with_pose>
   </link>

Commit message: update

File: balboa_description/urdf/balboa.urdf.xacro (robot description, xacro)
@@ -14,8 +14,8 @@
   <xacro:property name="wheel_width" value="${0.1*cm2m}" />
   <xacro:property name="encoder_resolution" value="1440" />
-  <xacro:property name="vel_update_rate" value="10" />
+  <xacro:property name="vel_update_rate" value="500" />
   <link name="origin_link" />
   <joint name="origin_joint" type="fixed">
-    <origin xyz="0 0 ${wheel_radius - wheel_z_offset}" rpy="0 0 0"/>
+    <origin xyz="0 0 ${wheel_radius - wheel_z_offset}" rpy="0.0 ${10*deg2rad} 0.0"/>
     <parent link="origin_link"/>
     <child link="base_link"/>
@@ -24,5 +24,4 @@
   <link name="base_link">
     <visual>
-      <origin xyz="0 0 0" rpy="0 ${0*deg2rad} 0"/>
       <geometry>
         <mesh filename="file://$(find balboa_description)/meshes/body.stl" />
@@ -30,5 +29,4 @@
     </visual>
     <collision name="balboa_collision">
-      <origin xyz="0 0 0" rpy="0 0 0"/>
       <geometry>
         <mesh filename="file://$(find balboa_description)/meshes/body.stl" />
@@ -36,5 +34,5 @@
     </collision>
     <xacro:inertial_cuboid_with_pose mass="1.0" x="${body_x}" y="${body_y}" z="${body_z}">
-      <origin xyz="${body_x/2} ${body_y/2} ${body_z/2}" />
+      <origin xyz="0.0 0.0 ${body_z/2}" />
       <!-- <origin xyz="0 0 0" /> -->
     </xacro:inertial_cuboid_with_pose>

Commit message: balboa balancing itself

File: balboa_description/urdf/balboa.urdf.xacro (robot description, xacro)
@@ -14,8 +14,8 @@
   <xacro:property name="wheel_width" value="${0.1*cm2m}" />
   <xacro:property name="encoder_resolution" value="1440" />
-  <xacro:property name="vel_update_rate" value="500" />
+  <xacro:property name="vel_update_rate" value="100" />
   <link name="origin_link" />
   <joint name="origin_joint" type="fixed">
-    <origin xyz="0 0 ${wheel_radius - wheel_z_offset}" rpy="0.0 ${10*deg2rad} 0.0"/>
+    <origin xyz="0 0 ${wheel_radius - wheel_z_offset}" rpy="0.0 ${5*deg2rad} 0.0"/>
     <parent link="origin_link"/>
     <child link="base_link"/>

Commit message: not using Twist anymore

File: balboa_description/urdf/balboa.urdf.xacro (robot description, xacro)
@@ -17,5 +17,5 @@
   <link name="origin_link" />
   <joint name="origin_joint" type="fixed">
-    <origin xyz="0 0 ${wheel_radius - wheel_z_offset}" rpy="0.0 ${5*deg2rad} 0.0"/>
+    <origin xyz="0 0 ${wheel_radius - wheel_z_offset}" rpy="0.0 0.0 0.0"/>
     <parent link="origin_link"/>
     <child link="base_link"/>
@@ -81,5 +81,5 @@
   </xacro:wheel>
   <!-- Ground truth pose -->
-  <gazebo>
+  <!-- <gazebo>
     <plugin name="gazebo_ros_p3d_robot" filename="libgazebo_ros_p3d.so">
       <ros>
@@ -94,4 +94,4 @@
       <gaussian_noise>0.0</gaussian_noise>
     </plugin>
-  </gazebo>
+  </gazebo> -->
 </robot>
